Commit message: assign limits

File: eggs_machina/model/meshes/assembly.urdf (robot description, URDF)
Before this commit: robot assembly, 5 links, 4 joints
Joints:
- joint Revolute-rob1: limit lower=0 upper=0 effort=80 velocity=5 -> lower=0 upper=6 effort=80 velocity=5
- joint Revolute-rob2: limit lower=0 upper=0 effort=80 velocity=5 -> lower=0 upper=6 effort=80 velocity=5
- joint Revolute-rob3: limit lower=0 upper=0 effort=80 velocity=5 -> lower=0 upper=6 effort=80 velocity=5
